Commit message: Changed sonar orientation

File: xacro/base_car_sonar.xacro (robot description, xacro)
@@ -67,5 +67,5 @@
     </link>
     <joint name="${namespace}/test_joint" type="revolute">
-      <origin xyz="0 0 3" rpy="0 ${pi/2} ${pi/2}"/>
+      <origin xyz="0 0 0.5" rpy="0 0 ${pi/2}"/>
       <parent link="${namespace}/base_link" />
       <child link="${namespace}/test_link" />
